File: VasulkaTranslocationPCB/VasulkaTranslocationPCB.kicad_pcb (KiCad board)
At the start: 2 copper layers, 243.8 x 332.7 mm, 280 parts, among them J1 Barrel_Jack, J2 BULB-, J3 BULB+, Q1 IRF510, Q10 IRF510, Q11 IRF510, Q12 IRF510, Q13 IRF510, Q14 IRF510, Q15 IRF510, Q16 IRF510, Q17 IRF510, Q18 IRF9520, Q19 IRF9520, Q2 IRF510, Q20 IRF9520, Q21 2N3904, Q22 2N3904, Q23 2N3904, Q24 IRF9520, Q25 IRF9520, Q26 IRF9520, Q27 2N3904, Q28 2N3904, Q29 2N3904, Q3 IRF510, Q30 IRF9520, Q31 IRF9520, Q32 2N3904, Q33 2N3904, Q34 IRF9520, Q35 IRF9520, Q36 IRF9520, Q37 2N3904, Q38 2N3904, Q39 2N3904, Q4 IRF510, Q40 IRF9520, Q41 IRF9520, Q42 IRF9520, Q43 2N3904, Q44 2N3904, Q45 2N3904, Q46 IRF9520, Q47 IRF9520, Q48 IRF9520, Q49 2N3904, Q5 IRF510, Q50 2N3904, Q51 2N3904, Q6 IRF510, Q7 IRF510, Q8 IRF510, Q9 IRF510, U1 TEENSY_3.5, U10 VO618A-4, U11 VO618A-4, U12 VO618A-4, U13 VO618A-4, U14 VO618A-4, U15 VO618A-4, U16 VO618A-4, U17 VO618A-4, U18 VO618A-4, U19 VO618A-4, U2 VO618A-4, U20 VO618A-4, U21 VO618A-4, U22 VO618A-4, U23 VO618A-4, U24 VO618A-4, U25 VO618A-4, U26 VO618A-4, U27 VO618A-4, U28 VO618A-4, U29 VO618A-4, U3 VO618A-4, U30 VO618A-4, U31 VO618A-4, U32 VO618A-4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

Commit message: CHANGED graphics
Other:
- board text added: "***K. DANAE KEILMAN//09/29/19//V1.0***"
- board text added: "THE BROTHERHOOD TRANSLOCATIONS Woody Vasulka VASULKA.ORG"
- board text removed: "K. DANAE KEILMAN TRANSLOCATION 09/29/19 V1.0"
Changed lines of the file:
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@@
-(kicad_pcb (version 20171130) (host pcbnew "(5.0.0-3-g5ebb6b6)")
+(kicad_pcb (version 20171130) (host pcbnew "(5.1.5-0-10_14)")
   (general
     (thickness 1.6)
-    (drawings 46)
+    (drawings 47)
     (tracks 1214)
     (zones 0)
@@
     (zone_45_only no)
     (trace_min 0.2)
-    (segment_width 0.2)
-    (edge_width 0.2)
     (via_size 0.8)
     (via_drill 0.4)
@@
     (uvia_min_size 0.2)
     (uvia_min_drill 0.1)
+    (edge_width 0.2)
+    (segment_width 0.2)
     (pcb_text_width 0.3)
     (pcb_text_size 1.5 1.5)
@@
     (mod_text_size 1 1)
     (mod_text_width 0.15)
-    (pad_size 1.524 1.524)
-    (pad_drill 0.762)
+    (pad_size 3.175 3.175)
+    (pad_drill 1.778)
     (pad_to_mask_clearance 0.2)
     (aux_axis_origin 0 0)
@@
       (linewidth 0.100000)
       (plotframeref false)
-      (viasonmask false)
+      (viasonmask true)
       (mode 1)
       (useauxorigin false)
@@
       (plotvalue true)
       (plotinvisibletext false)
-      (padsonsilk false)
+      (padsonsilk true)
       (subtractmaskfromsilk false)
       (outputformat 1)
@@
     (tags "mounting hole 3.2mm no annular m3")
     (attr virtual)
-    (fp_text reference MH2 (at 0 -4.2) (layer F.SilkS)
+    (fp_text reference MH2 (at 0 -4.2) (layer Dwgs.User)
       (effects (font (size 1 1) (thickness 0.15)))
     )
@@
     (tags "mounting hole 3.2mm no annular m3")
     (attr virtual)
-    (fp_text reference MH1 (at 0 -4.2) (layer F.SilkS)
+    (fp_text reference MH1 (at 0 -4.2) (layer Dwgs.User)
       (effects (font (size 1 1) (thickness 0.15)))
     )
@@
     (tags "mounting hole 3.2mm no annular m3")
     (attr virtual)
-    (fp_text reference MH3 (at 0 -4.2) (layer F.SilkS)
+    (fp_text reference MH3 (at 0 -4.2) (layer Dwgs.User)
       (effects (font (size 1 1) (thickness 0.15)))
     )
@@
     (tags "mounting hole 3.2mm no annular m3")
     (attr virtual)
-    (fp_text reference MH4 (at 0 -4.2) (layer F.SilkS)
+    (fp_text reference MH4 (at 0 -4.2) (layer Dwgs.User)
       (effects (font (size 1 1) (thickness 0.15)))
     )
@@
     (pad 1 np_thru_hole circle (at 0 0) (size 3.2 3.2) (drill 3.2) (layers *.Cu *.Mask))
   )
+  (gr_text "THE BROTHERHOOD\nTRANSLOCATIONS\nWoody Vasulka\nVASULKA.ORG" (at 337.185 196.85 90) (layer F.SilkS)
+    (effects (font (size 3 3) (thickness 0.45)))
+  )
   (dimension 243.84 (width 0.3) (layer F.SilkS)
     (gr_text "243.840 mm" (at 228.6 451.045) (layer F.SilkS)
@@
     (effects (font (size 5 5) (thickness 0.6)))
   )
-  (gr_text "K. DANAE KEILMAN\nTRANSLOCATION\n09/29/19\nV1.0" (at 128.905 161.925 90) (layer B.SilkS)
-    (effects (font (size 5 5) (thickness 1)) (justify mirror))
+  (gr_text "***K. DANAE KEILMAN//09/29/19//V1.0***" (at 108.585 145.415 90) (layer B.Cu)
+    (effects (font (size 1.5 1.5) (thickness 0.3)) (justify mirror))
   )
   (segment (start 212.725 177.9905) (end 209.55 181.1655) (width 0.25) (layer F.Cu) (net 11))
@@
     (polygon
       (pts
-        (xy 106.68 426.72) (xy 119.38 426.72) (xy 119.38 439.42) (xy 337.82 439.42) (xy 337.82 426.72)
+        (xy 111.125 426.085) (xy 119.38 426.72) (xy 119.38 439.42) (xy 337.82 439.42) (xy 337.82 426.72)
         (xy 350.52 426.72) (xy 350.52 119.38) (xy 337.82 119.38) (xy 337.82 106.68) (xy 119.38 106.68)
-        (xy 119.38 119.38) (xy 106.68 119.38)
+        (xy 119.38 119.38) (xy 111.125 118.745)
       )
     )
